File: Solder.kicad_pcb (KiCad board)
At the start: 2 copper layers, 60.6 x 72.3 mm, 13 parts, among them Q1 NPN, Q2 NPN, Q3 NPN, Q4 NPN, SW1 SW_Push, SW2 SW_Push

Commit message: added logos to the back
Parts:
- R1, R2, R3, R4, R6: value R 1k -> R 220
